File: schematic/Kopplingsschema.sch (EAGLE design)
At the start: 6 parts

Commit message: Updated schematic
Connections:
- new net ICSPCLK: PIC16F15344.18
- new net ICSPDAT: PIC16F15344.19
- new net VPP: PIC16F15344.4
- net 3.3V: now also PIC16F15344.1
- net BT-RX: now also PIC16F15344.11
- net BT-TX: now also PIC16F15344.12
- net GND: now also PIC16F15344.20
- net GPS-RX: now also PIC16F15344.6
- net GPS-TX: now also PIC16F15344.5
- net GSM-RX: now also PIC16F15344.15
- net GSM-TX: now also PIC16F15344.16
- net SIGFOX-RX: now also PIC16F15344.8
- net SIGFOX-TX: now also PIC16F15344.7
- net WIFI-RX: now also PIC16F15344.3
- net WIFI-TX: now also PIC16F15344.2
Changed lines of the file:
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@@
 <label x="-22.86" y="7.62" size="1.778" layer="95" rot="R180" xref="yes"/>
+</segment>
+<segment>
+<pinref part="PIC16F15344" gate="G$1" pin="2"/>
+<wire x1="-96.52" y1="63.5" x2="-111.76" y2="63.5" width="0.1524" layer="91"/>
+<label x="-111.76" y="63.5" size="1.778" layer="95" rot="R180" xref="yes"/>
 </segment>
 </net>
@@
 <label x="78.74" y="-55.88" size="1.778" layer="95" rot="R270" xref="yes"/>
 </segment>
+<segment>
+<pinref part="PIC16F15344" gate="G$1" pin="1"/>
+<wire x1="-96.52" y1="66.04" x2="-99.06" y2="66.04" width="0.1524" layer="91"/>
+<label x="-99.06" y="66.04" size="1.778" layer="95" rot="R180" xref="yes"/>
+</segment>
 </net>
 <net name="GND" class="0">
@@
 <label x="-86.36" y="-40.64" size="1.778" layer="95" rot="R270" xref="yes"/>
 </segment>
+<segment>
+<pinref part="PIC16F15344" gate="G$1" pin="20"/>
+<wire x1="-81.28" y1="66.04" x2="-78.74" y2="66.04" width="0.1524" layer="91"/>
+<label x="-78.74" y="66.04" size="1.778" layer="95" xref="yes"/>
+</segment>
 </net>
 <net name="WIFI-RX" class="0">
@@
 <label x="20.32" y="-7.62" size="1.778" layer="95" xref="yes"/>
 </segment>
+<segment>
+<pinref part="PIC16F15344" gate="G$1" pin="3"/>
+<wire x1="-96.52" y1="60.96" x2="-99.06" y2="60.96" width="0.1524" layer="91"/>
+<label x="-99.06" y="60.96" size="1.778" layer="95" rot="R180" xref="yes"/>
+</segment>
 </net>
 <net name="5V" class="0">
@@
 <label x="25.4" y="50.8" size="1.778" layer="95" xref="yes"/>
 </segment>
+<segment>
+<pinref part="PIC16F15344" gate="G$1" pin="15"/>
+<wire x1="-81.28" y1="53.34" x2="-66.04" y2="53.34" width="0.1524" layer="91"/>
+<label x="-66.04" y="53.34" size="1.778" layer="95" xref="yes"/>
+</segment>
 </net>
 <net name="GSM-TX" class="0">
@@
 <label x="25.4" y="45.72" size="1.778" layer="95" xref="yes"/>
 </segment>
+<segment>
+<pinref part="PIC16F15344" gate="G$1" pin="16"/>
+<wire x1="-81.28" y1="55.88" x2="-78.74" y2="55.88" width="0.1524" layer="91"/>
+<label x="-78.74" y="55.88" size="1.778" layer="95" xref="yes"/>
+</segment>
 </net>
 <net name="GPS-TX" class="0">
@@
 <label x="73.66" y="20.32" size="1.778" layer="95" rot="R270" xref="yes"/>
 </segment>
+<segment>
+<pinref part="PIC16F15344" gate="G$1" pin="5"/>
+<wire x1="-96.52" y1="55.88" x2="-99.06" y2="55.88" width="0.1524" layer="91"/>
+<label x="-99.06" y="55.88" size="1.778" layer="95" rot="R180" xref="yes"/>
+</segment>
 </net>
 <net name="GPS-RX" class="0">
@@
 <label x="78.74" y="20.32" size="1.778" layer="95" rot="R270" xref="yes"/>
 </segment>
+<segment>
+<pinref part="PIC16F15344" gate="G$1" pin="6"/>
+<wire x1="-96.52" y1="53.34" x2="-116.84" y2="53.34" width="0.1524" layer="91"/>
+<label x="-116.84" y="53.34" size="1.778" layer="95" rot="R180" xref="yes"/>
+</segment>
 </net>
 <net name="SIGFOX-TX" class="0">
@@
 <label x="63.5" y="-55.88" size="1.778" layer="95" rot="R180" xref="yes"/>
 </segment>
+<segment>
+<pinref part="PIC16F15344" gate="G$1" pin="7"/>
+<wire x1="-96.52" y1="50.8" x2="-99.06" y2="50.8" width="0.1524" layer="91"/>
+<label x="-99.06" y="50.8" size="1.778" layer="95" rot="R180" xref="yes"/>
+</segment>
 </net>
 <net name="SIGFOX-RX" class="0">
@@
 <label x="66.04" y="-55.88" size="1.778" layer="95" rot="R270" xref="yes"/>
 </segment>
+<segment>
+<pinref part="PIC16F15344" gate="G$1" pin="8"/>
+<wire x1="-96.52" y1="48.26" x2="-116.84" y2="48.26" width="0.1524" layer="91"/>
+<label x="-116.84" y="48.26" size="1.778" layer="95" rot="R180" xref="yes"/>
+</segment>
 </net>
 <net name="BT-TX" class="0">
@@
 <label x="-81.28" y="-40.64" size="1.778" layer="95" rot="R270" xref="yes"/>
 </segment>
+<segment>
+<pinref part="PIC16F15344" gate="G$1" pin="12"/>
+<wire x1="-81.28" y1="45.72" x2="-78.74" y2="45.72" width="0.1524" layer="91"/>
+<label x="-78.74" y="45.72" size="1.778" layer="95" xref="yes"/>
+</segment>
 </net>
 <net name="BT-RX" class="0">
@@
 <label x="-76.2" y="-40.64" size="1.778" layer="95" rot="R270" xref="yes"/>
 </segment>
-</net>
+<segment>
+<pinref part="PIC16F15344" gate="G$1" pin="11"/>
+<wire x1="-81.28" y1="43.18" x2="-68.58" y2="43.18" width="0.1524" layer="91"/>
+<label x="-68.58" y="43.18" size="1.778" layer="95" xref="yes"/>
+</segment>
+</net>
+<net name="VPP" class="0">
+<segment>
+<pinref part="PIC16F15344" gate="G$1" pin="4"/>
+<wire x1="-96.52" y1="58.42" x2="-111.76" y2="58.42" width="0.1524" layer="91"/>
+<label x="-111.76" y="58.42" size="1.778" layer="95" rot="R180" xref="yes"/>
+</segment>
+</net>
+<net name="ICSPDAT" class="0">
+<segment>
+<pinref part="PIC16F15344" gate="G$1" pin="19"/>
+<wire x1="-81.28" y1="63.5" x2="-63.5" y2="63.5" width="0.1524" layer="91"/>
+<label x="-63.5" y="63.5" size="1.778" layer="95" xref="yes"/>
+</segment>
+</net>
+<net name="ICSPCLK" class="0">
+<segment>
+<pinref part="PIC16F15344" gate="G$1" pin="18"/>
+<wire x1="-81.28" y1="60.96" x2="-78.74" y2="60.96" width="0.1524" layer="91"/>
+<label x="-78.74" y="60.96" size="1.778" layer="95" xref="yes"/>
+</segment>
+</net>
